File: pcb/ya36.kicad_pcb (KiCad board)
At the start: 2 copper layers, 225 x 67 mm, 92 parts, among them J1 MJ-4PP-9, J2 MJ-4PP-9, SW1 SW_PUSH, SW10 SW_PUSH, SW11 SW_PUSH, SW12 SW_PUSH, SW13 SW_PUSH, SW14 SW_PUSH, SW15 SW_PUSH, SW16 SW_PUSH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

Commit message: Update gbr
Routing:
- net ROW4: track 78.4 -> 64.0 mm
- net ROW4R: track 61.8 -> 60.6 mm
